Commit message: 完善了一下下

File: src/robot_description/urdf/robot/actuator/caster.urdf.xacro (robot description, xacro)
@@ -1,5 +1,5 @@
 <?xml version="1.0"?>
 <!-- 万相轮 -->
-<robot xmlns:xacro="http://www.ros.org/wiki/xacro">
+<robot xmlns:xacro="http://ros.org/wiki/xacro">
    <xacro:include filename="$(find robot_description)/urdf/robot/common_inertia.xacro" />
     <xacro:macro name="caster_xacro" params="caster_name xyz">

File: src/robot_description/urdf/robot/actuator/wheel.urdf.xacro (robot description, xacro)
@@ -1,5 +1,5 @@
 <?xml version="1.0"?>
 <!-- 轮子 -->
-<robot xmlns:xacro="http://www.ros.org/wiki/xacro">
+<robot xmlns:xacro="http://ros.org/wiki/xacro">
    <xacro:include filename="$(find robot_description)/urdf/robot/common_inertia.xacro" />
     <xacro:macro name="wheel_xacro" params="wheel_name xyz">
@@ -38,4 +38,5 @@
             <origin xyz="${xyz}" />
             <axis xyz="0 1 0" />
+            <dynamics damping="0.2" friction="0.02" />
         </joint>
     </xacro:macro>

File: src/robot_description/urdf/robot/base.urdf.xacro (robot description, xacro)
@@ -1,7 +1,7 @@
 <?xml version="1.0"?>
-<robot xmlns:xacro="http://www.ros.org/wiki/xacro">
+<robot xmlns:xacro="http://ros.org/wiki/xacro">
    <xacro:include filename="$(find robot_description)/urdf/robot/common_inertia.xacro" />
     <xacro:macro name="base_xacro" params="length radius">
-     <link name="base_footprint" />
+        <link name="base_footprint" />
         <joint name="base_joint" type="fixed">
             <parent link="base_footprint" />

File: src/robot_description/urdf/robot/robot.urdf.xacro (robot description, xacro)
@@ -1,28 +1,28 @@
 <?xml version="1.0"?>
-<robot xmlns:xacro="http://www.ros.org/wiki/xacro" name="robot">
-    <xacro:include filename="$(find robot_description)/urdf/robot/base.urdf.xacro" />
-    <!-- 传感器组件 -->
-    <xacro:include filename="$(find robot_description)/urdf/robot/sensor/imu.urdf.xacro" />
-    <xacro:include filename="$(find robot_description)/urdf/robot/sensor/laser.urdf.xacro" />
-    <xacro:include filename="$(find robot_description)/urdf/robot/sensor/camera.urdf.xacro" />
-     <!-- 执行器组件 -->
-    <xacro:include filename="$(find robot_description)/urdf/robot/actuator/wheel.urdf.xacro" />
-    <xacro:include filename="$(find robot_description)/urdf/robot/actuator/caster.urdf.xacro" />
-    <xacro:base_xacro length="0.12" radius="0.1" />
-    <!-- 传感器 -->
-    <xacro:imu_xacro xyz="0 0 0.02" />
-    <xacro:laser_xacro xyz="0 0 0.10" />
-    <xacro:camera_xacro xyz="0.10 0 0.075" />
-    <!-- 执行器主动轮+从动轮 -->
-    <xacro:wheel_xacro wheel_name="left" xyz="0 0.10 -0.06" />
-    <xacro:wheel_xacro wheel_name="right" xyz="0 -0.10 -0.06" />
-    <xacro:caster_xacro caster_name="front" xyz="0.08 0.0 -0.076" />
-    <xacro:caster_xacro caster_name="back" xyz="-0.08 0.0 -0.076" />
-    <!-- Gazebo 插件 -->
-    <xacro:include filename="$(find robot_description)/urdf/robot/plugins/gazebo_control_plugin.xacro" />
-    <!-- <xacro:gazebo_control_plugin /> -->
-    <xacro:include filename="$(find robot_description)/urdf/robot/robot.ros2_control.xacro" />
-    <xacro:robot_ros2_control />
-    <xacro:include filename="$(find robot_description)/urdf/robot/plugins/gazebo_sensor_plugin.xacro" />
-    <xacro:gazebo_sensor_plugin />
+<robot name="robot" xmlns:xacro="http://ros.org/wiki/xacro">
+    <!-- 定义机器人 -->
+    <xacro:macro name="robot">
+        <xacro:include filename="$(find robot_description)/urdf/robot/base.urdf.xacro" />
+        <!-- 传感器组件 -->
+        <xacro:include filename="$(find robot_description)/urdf/robot/sensor/imu.urdf.xacro" />
+        <xacro:include filename="$(find robot_description)/urdf/robot/sensor/laser.urdf.xacro" />
+        <xacro:include filename="$(find ros2_livox_simulation)/urdf/mid360.xacro" />
+        <xacro:include filename="$(find robot_description)/urdf/robot/sensor/camera.urdf.xacro" />
+         <!-- 执行器组件 -->
+        <xacro:include filename="$(find robot_description)/urdf/robot/actuator/wheel.urdf.xacro" />
+        <xacro:include filename="$(find robot_description)/urdf/robot/actuator/caster.urdf.xacro" />
+        <!-- 底盘 -->
+        <xacro:base_xacro length="0.12" radius="0.1" />
+        <!-- 传感器 -->
+        <xacro:imu_xacro parent="base_link" xyz="0 0 0.02" />
+        <xacro:laser_xacro parent="base_link" xyz="0 0 0.10" />
+        <xacro:camera_xacro parent="base_link" xyz="0.10 0 0.075" />
+        <!-- 执行器主动轮+从动轮 -->
+        <xacro:wheel_xacro wheel_name="left" xyz="0 0.10 -0.06" />
+        <xacro:wheel_xacro wheel_name="right" xyz="0 -0.10 -0.06" />
+        <xacro:caster_xacro caster_name="front" xyz="0.08 0.0 -0.076" />
+        <xacro:caster_xacro caster_name="back" xyz="-0.08 0.0 -0.076" />
+    </xacro:macro>
+    <!-- 实例化机器人 -->
+    <xacro:robot />
 </robot>

File: src/robot_description/urdf/robot/sensor/camera.urdf.xacro (robot description, xacro)
@@ -1,7 +1,7 @@
 <?xml version="1.0"?>
 <!-- 相机 -->
-<robot xmlns:xacro="http://www.ros.org/wiki/xacro">
+<robot xmlns:xacro="http://ros.org/wiki/xacro">
    <xacro:include filename="$(find robot_description)/urdf/robot/common_inertia.xacro" />
-    <xacro:macro name="camera_xacro" params="xyz">
+    <xacro:macro name="camera_xacro" params="parent xyz">
         <link name="camera_link">
             <visual>
@@ -34,5 +34,5 @@
         <!-- 机器人关节 -->
         <joint name="camera_joint" type="fixed">
-            <parent link="base_link" />
+            <parent link="${parent}" />
             <child link="camera_link" />
             <origin xyz="${xyz}" />

File: src/robot_description/urdf/robot/sensor/imu.urdf.xacro (robot description, xacro)
@@ -1,7 +1,7 @@
 <?xml version="1.0"?>
 <!-- imu -->
-<robot xmlns:xacro="http://www.ros.org/wiki/xacro">
-   <xacro:include filename="$(find robot_description)/urdf/robot/common_inertia.xacro" />
-    <xacro:macro name="imu_xacro" params="xyz">
+<robot xmlns:xacro="http://ros.org/wiki/xacro">
+    <xacro:include filename="$(find robot_description)/urdf/robot/common_inertia.xacro" />
+    <xacro:macro name="imu_xacro" params="parent xyz">
         <link name="imu_link">
             <visual>
@@ -27,5 +27,5 @@
         <!-- 机器人关节 -->
         <joint name="imu_joint" type="fixed">
-            <parent link="base_link" />
+            <parent link="${parent}" />
             <child link="imu_link" />
             <origin xyz="${xyz}" />

File: src/robot_description/urdf/robot/sensor/laser.urdf.xacro (robot description, xacro)
@@ -1,7 +1,7 @@
 <?xml version="1.0"?>
 <!-- 雷达 -->
-<robot xmlns:xacro="http://www.ros.org/wiki/xacro">
+<robot xmlns:xacro="http://ros.org/wiki/xacro">
    <xacro:include filename="$(find robot_description)/urdf/robot/common_inertia.xacro" />
-    <xacro:macro name="laser_xacro" params="xyz">
+    <xacro:macro name="laser_xacro" params="parent xyz">
         <gazebo reference="laser_cylinder_link">
             <material>Gazebo/Black</material>
@@ -56,5 +56,5 @@
         <!-- 雷达支撑杆关节 -->
         <joint name="laser_cylinder_joint" type="fixed">
-            <parent link="base_link" />
+            <parent link="${parent}" />
             <child link="laser_cylinder_link" />
             <origin xyz="${xyz}" />
